Commit message: all fixed

File: hunter_description/urdf/vehicle.xacro (robot description, xacro)
@@ -85,5 +85,5 @@
   <joint
     name="front_steer_left_joint"
-    type="revolute">
+    type="fixed">
     <origin
       xyz="0.37142 0.29199 -0.1955"
@@ -93,5 +93,5 @@
     <child
       link="front_steer_left_link" />
-    <axis
+    <!-- <axis
       xyz="0 1 0" />
     <limit
@@ -99,5 +99,5 @@
       upper="0.69"
       effort="0"
-      velocity="0" />
+      velocity="0" /> -->
   </joint>
   <link
@@ -143,5 +143,5 @@
   <joint
     name="front_left_wheel_joint"
-    type="continuous">
+    type="fixed">
     <origin
       xyz="0 0 0"
@@ -151,6 +151,6 @@
     <child
       link="front_left_wheel_link" />
-    <axis
-      xyz="0 0 -1" />
+    <!-- <axis
+      xyz="0 0 -1" /> -->
   </joint>
   <link
@@ -194,5 +194,5 @@
   <joint
     name="front_steer_right_joint"
-    type="revolute">
+    type="fixed">
     <origin
       xyz="0.37142 -0.29201 -0.1955"
@@ -202,5 +202,5 @@
     <child
       link="front_steer_right_link" />
-    <axis
+    <!-- <axis
       xyz="0 1 0" />
     <limit
@@ -208,5 +208,5 @@
       upper="0.69"
       effort="0"
-      velocity="0" />
+      velocity="0" /> -->
   </joint>
   <link
@@ -252,5 +252,5 @@
   <joint
     name="front_right_wheel_joint"
-    type="continuous">
+    type="fixed">
     <origin
       xyz="0 0 0"
@@ -260,6 +260,6 @@
     <child
       link="front_right_wheel_link" />
-    <axis
-      xyz="0 0 -1" />
+    <!-- <axis
+      xyz="0 0 -1" /> -->
   </joint>
   <link
@@ -305,5 +305,5 @@
   <joint
     name="left_rear_joint"
-    type="continuous">
+    type="fixed">
     <origin
       xyz="-0.28 0.29249 -0.19558"
@@ -313,11 +313,11 @@
     <child
       link="left_rear_link" />
-    <axis
-      xyz="0 0 -1" />
-    <limit
+    <!-- <axis
+      xyz="0 0 -1" /> -->
+    <!-- <limit
       lower="-3.14"
       upper="3.14"
       effort="0"
-      velocity="0" />
+      velocity="0" /> -->
   </joint>
   <link
@@ -363,5 +363,5 @@
   <joint
     name="right_rear_joint"
-    type="continuous">
+    type="fixed">
     <origin
       xyz="-0.28018 -0.29251 -0.19558"
@@ -371,5 +371,5 @@
     <child
       link="right_rear_link" />
-    <axis
+    <!-- <axis
       xyz="0 0 -1" />
     <limit
@@ -377,5 +377,5 @@
       upper="3.14"
       effort="0"
-      velocity="0" />
+      velocity="0" /> -->
   </joint>
   <link
@@ -419,5 +419,5 @@
   <joint
     name="front_steer_joint"
-    type="revolute">
+    type="fixed">
     <origin
       xyz="0.44792 -1.1431E-05 -0.121"
@@ -427,5 +427,5 @@
     <child
       link="front_steer_link" />
-    <axis
+    <!-- <axis
       xyz="0 0 1" />
     <limit
@@ -433,5 +433,5 @@
       upper="0.72"
       effort="0"
-      velocity="0" />
+      velocity="0" /> -->
   </joint>
   <link
@@ -475,5 +475,5 @@
   <joint
     name="rear_wheel_joint"
-    type="continuous">
+    type="fixed">
     <origin
       xyz="-0.42408 -1.1431E-05 -0.085581"
@@ -483,6 +483,6 @@
     <child
       link="rear_wheel_link" />
-    <axis
-      xyz="0 0 1" />
+    <!-- <axis
+      xyz="0 0 1" /> -->
   </joint>
   <link
